File: pcb/control_board_1/control_board_1.kicad_sch (KiCad schematic)
At the start: 5 parts, among them J2 JST4 Power, SW1 Mode Switch

Commit message: JLCPCB has violated me
Parts:
- removed H1: HUB75 Connector, symbol lightslop2:hub75_din_connector
- removed J2: JST4 Power, symbol lightslop2:jst4_vh_3.96_power
- removed SD: Adafruit MicroSD Adapter, symbol lightslop2:usd_breakout_adafruit
- added H2: HUB75 Data, Connector_IDC:IDC-Header_2x08_P2.54mm_Vertical, symbol overblinking:hub75_din_connector
- added J1: JST4 VH Power, Connector_JST:JST_VH_B4PS-VH_1x04_P3.96mm_Horizontal, symbol overblinking:jst4_vh_3.96_power
- added SD1: 4682 SD Adapter, overblinking:usd_breakout_adafruit, symbol overblinking:usd_breakout_adafruit
- SW1: footprint (none) -> Button_Switch_THT:SW_PUSH_6mm
Connections:
- net 3V3: now also SD1.1 (3V)
- net 5V: now also J1.1 (VIN), J1.2 (VIN)
- net A: now also H2.9 (A)
- net B: now also H2.10 (B)
- net B0: now also H2.3 (B0)
- net B1: now also H2.7 (B1)
- net C: now also H2.11 (C)
- net CD: now also SD1.9 (CD)
- net CLK: now also H2.13 (CLK)
- net CS: now also SD1.6 (CS)
- net D: now also H2.12 (D)
- net E: now also H2.8 (E)
- net G0: now also H2.2 (G0)
- net G1: now also H2.6 (G1)
- net GND: now also H2.16 (GND), H2.4 (GND), J1.3 (GND), J1.4 (GND), SD1.2 (GND)
- net LATCH: now also H2.14 (OEN)
- net MISO: now also SD1.4 (MISO)
- net MOSI: now also SD1.5 (MOSI)
- net OEN: now also H2.15 (OEN)
- net R0: now also H2.1 (R0)
- net R1: now also H2.5 (R1)
- net SCLK: now also SD1.3 (CLK)
- no-connect marks 0 -> 13
Changed lines of the file:
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@@
 		(color 0 0 0 0)
 	)
+	(no_connect
+		(at 130.81 106.68)
+	)
+	(no_connect
+		(at 85.09 60.96)
+	)
+	(no_connect
+		(at 130.81 86.36)
+	)
+	(no_connect
+		(at 181.61 85.09)
+	)
+	(no_connect
+		(at 85.09 63.5)
+	)
+	(no_connect
+		(at 130.81 83.82)
+	)
+	(no_connect
+		(at 130.81 99.06)
+	)
+	(no_connect
+		(at 130.81 101.6)
+	)
+	(no_connect
+		(at 107.95 45.72)
+	)
+	(no_connect
+		(at 85.09 106.68)
+	)
+	(no_connect
+		(at 130.81 96.52)
+	)
+	(no_connect
+		(at 130.81 91.44)
+	)
+	(no_connect
+		(at 181.61 82.55)
+	)
 	(wire
 		(pts
@@
 	)
 	(symbol
-		(lib_id "lightslop2:usd_breakout_adafruit")
+		(lib_id "overblinking:usd_breakout_adafruit")
 		(at 190.5 71.12 270)
 		(unit 1)
@@
 		(dnp no)
 		(fields_autoplaced yes)
-		(property "Reference" "SD"
-			(at 205.994 77.216 0)
-			(effects
-				(font
-					(size 1.27 1.27)
-				)
-			)
-		)
-		(property "Value" "Adafruit MicroSD Adapter"
-			(at 203.708 77.47 0)
-			(effects
-				(font
-					(size 1.27 1.27)
-				)
-			)
-		)
-		(property "Footprint" ""
+		(property "Reference" "SD1"
+			(at 203.2 76.1999 90)
+			(effects
+				(font
+					(size 1.27 1.27)
+				)
+				(justify left)
+			)
+		)
+		(property "Value" "4682 SD Adapter"
+			(at 203.2 78.7399 90)
+			(effects
+				(font
+					(size 1.27 1.27)
+				)
+				(justify left)
+			)
+		)
+		(property "Footprint" "overblinking:usd_breakout_adafruit"
 			(at 190.5 71.12 0)
 			(effects
@@
 			)
 		)
+		(pin "4"
+		)
+		(pin "7"
+		)
+		(pin "8"
+		)
+		(pin "3"
+		)
 		(pin "1"
 		)
-		(pin "3"
+		(pin "5"
 		)
 		(pin "2"
 		)
-		(pin "5"
-		)
 		(pin "6"
 		)
-		(pin "7"
-		)
-		(pin "8"
-		)
 		(pin "9"
-		)
-		(pin "4"
 		)
 		(instances
 			(project "control_board_1"
 				(path "/c74dadd3-b9fd-4089-b688-07ec3572b669"
-					(reference "SD")
+					(reference "SD1")
 					(unit 1)
 				)
@@
 	)
 	(symbol
-		(lib_id "lightslop2:hub75_din_connector")
+		(lib_id "overblinking:jst4_vh_3.96_power")
+		(at 67.31 161.29 270)
+		(unit 1)
+		(exclude_from_sim no)
+		(in_bom yes)
+		(on_board yes)
+		(dnp no)
+		(fields_autoplaced yes)
+		(property "Reference" "J1"
+			(at 55.245 147.32 90)
+			(effects
+				(font
+					(size 1.27 1.27)
+				)
+			)
+		)
+		(property "Value" "JST4 VH Power"
+			(at 55.245 149.86 90)
+			(effects
+				(font
+					(size 1.27 1.27)
+				)
+			)
+		)
+		(property "Footprint" "Connector_JST:JST_VH_B4PS-VH_1x04_P3.96mm_Horizontal"
+			(at 67.31 161.29 0)
+			(effects
+				(font
+					(size 1.27 1.27)
+				)
+				(hide yes)
+			)
+		)
+		(property "Datasheet" ""
+			(at 67.31 161.29 0)
+			(effects
+				(font
+					(size 1.27 1.27)
+				)
+				(hide yes)
+			)
+		)
+		(property "Description" ""
+			(at 67.31 161.29 0)
+			(effects
+				(font
+					(size 1.27 1.27)
+				)
+				(hide yes)
+			)
+		)
+		(pin "1"
+		)
+		(pin "3"
+		)
+		(pin "2"
+		)
+		(pin "4"
+		)
+		(instances
+			(project "control_board_1"
+				(path "/c74dadd3-b9fd-4089-b688-07ec3572b669"
+					(reference "J1")
+					(unit 1)
+				)
+			)
+		)
+	)
+	(symbol
+		(lib_id "overblinking:hub75_din_connector")
 		(at 189.23 109.22 0)
 		(unit 1)
@@
 		(dnp no)
 		(fields_autoplaced yes)
-		(property "Reference" "H1"
+		(property "Reference" "H2"
 			(at 192.405 106.68 0)
 			(effects
@@
 			)
 		)
-		(property "Value" "HUB75 Connector"
+		(property "Value" "HUB75 Data"
 			(at 192.405 109.22 0)
 			(effects
@@
 			)
 		)
-		(property "Footprint" ""
+		(property "Footprint" "Connector_IDC:IDC-Header_2x08_P2.54mm_Vertical"
 			(at 189.23 109.22 0)
 			(effects
@@
 			)
 		)
+		(pin "7"
+		)
+		(pin "10"
+		)
+		(pin "16"
+		)
 		(pin "2"
 		)
+		(pin "11"
+		)
+		(pin "9"
+		)
+		(pin "3"
+		)
 		(pin "4"
 		)
+		(pin "12"
+		)
+		(pin "14"
+		)
+		(pin "1"
+		)
+		(pin "5"
+		)
+		(pin "15"
+		)
 		(pin "6"
 		)
 		(pin "8"
 		)
-		(pin "12"
-		)
-		(pin "16"
-		)
-		(pin "11"
-		)
 		(pin "13"
-		)
-		(pin "15"
-		)
-		(pin "10"
-		)
-		(pin "14"
-		)
-		(pin "5"
-		)
-		(pin "7"
-		)
-		(pin "9"
-		)
-		(pin "3"
-		)
-		(pin "1"
 		)
 		(instances
 			(project "control_board_1"
 				(path "/c74dadd3-b9fd-4089-b688-07ec3572b669"
-					(reference "H1")
+					(reference "H2")
 					(unit 1)
 				)
@@
 			)
 		)
-		(property "Footprint" ""
+		(property "Footprint" "Button_Switch_THT:SW_PUSH_6mm"
 			(at 113.03 149.86 0)
 			(effects
@@
 					(unit 1)
 				)
-			)
-		)
-	)
-	(symbol
-		(lib_id "lightslop2:jst4_vh_3.96_power")
-		(at 67.31 161.29 270)
-		(unit 1)
-		(exclude_from_sim no)
-		(in_bom yes)
-		(on_board yes)
-		(dnp no)
-		(fields_autoplaced yes)
-		(property "Reference" "J2"
-			(at 55.245 147.32 90)
-			(effects
-				(font
-					(size 1.27 1.27)
-				)
-			)
-		)
-		(property "Value" "JST4 Power"
-			(at 55.245 149.86 90)
-			(effects
-				(font
-					(size 1.27 1.27)
-				)
-			)
-		)
-		(property "Footprint" ""
-			(at 67.31 161.29 0)
-			(effects
-				(font
-					(size 1.27 1.27)
-				)
-				(hide yes)
-			)
-		)
-		(property "Datasheet" ""
-			(at 67.31 161.29 0)
-			(effects
-				(font
-					(size 1.27 1.27)
-				)
-				(hide yes)
-			)
-		)
-		(property "Description" ""
-			(at 67.31 161.29 0)
-			(effects
-				(font
-					(size 1.27 1.27)
-				)
-				(hide yes)
-			)
-		)
-		(pin "1"
-		)
-		(pin "4"
-		)
-		(pin "3"
-		)
-		(pin "2"
-		)
-		(instances
-			(project "control_board_1"
-				(path "/c74dadd3-b9fd-4089-b688-07ec3572b669"
-					(reference "J2")
-					(unit 1)
-				)
